File: m0330.kicad_sch (KiCad schematic)
At the start: 246 parts, among them J2 Conn_01x04_MountingPin, J3 Conn_01x04_MountingPin, Q1 Q_PMOS_GSD AO3401A, Q2 Q_NMOS_GSD 2N7002, Q3 Q_NMOS_GSD 2N7002, Q4 2N3904, SW1 SW_Push, U1 XC6206P332MR, U2 74AHCT1G125, U3 STM32F411RETx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

Commit message: updates
Parts:
- SW1: footprint random-keyboard-parts:SKQG-1155865 -> controller:switch_K2-1187SQ-A4SW-06
Changed lines of the file:
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@@
       (effects (font (size 1.27 1.27)) (justify left))
     )
-    (property "Footprint" "random-keyboard-parts:SKQG-1155865" (at 63.5 112.395 0)
+    (property "Footprint" "controller:switch_K2-1187SQ-A4SW-06" (at 63.5 112.395 0)
       (effects (font (size 1.27 1.27)) hide)
     )
